File: SBCclock.kicad_pcb (KiCad board)
At the start: 4 copper layers, 37.5 x 23.4 mm, 20 parts, among them J1 Conn_01x07, J2 Conn_01x07, U1 74HCT14, U2 74HCT163, U3 74HCT112, U5 74HCT153, Y1 25.175MHz

Commit message: revise load capacitors
Parts:
- C1, C2: value 22pF -> 4.7pF
Changed lines of the file:
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@@
         (effects (font (size 1 1) (thickness 0.15)))
     )
-    (fp_text value "22pF" (at 0 1.68 90) (layer "F.Fab")
+    (fp_text value "4.7pF" (at 0 1.68 90) (layer "F.Fab")
         (effects (font (size 1 1) (thickness 0.15)))
     )
@@
         (effects (font (size 1 1) (thickness 0.15)) (justify mirror))
     )
-    (fp_text value "22pF" (at 0 -1.68) (layer "B.Fab")
-        (effects (font (size 1 1) (thickness 0.15)) (justify mirror))
-    )
+    (fp_text value "4.7pF" (at 0 -1.68) (layer "B.Fab")
+        (effects (font (size 1 1) (thickness 0.15)) (justify mirror))
+    )
